File: two_comparator_effect/two_comparator_effect.kicad_pcb (KiCad board)
At the start: 2 copper layers, 100 x 35 mm, 30 parts, among them J1 RCA, J2 RCA, J3 Barrel_Jack, Q1 2N3904, U1 LM311, U2 LM311, U3 LM311, U4 LM317

Commit message: updated two_comparator and added two_point_one
Parts:
- removed the U2 at (180.0, 70.0)
- removed U3: LM311, Package_DIP:DIP-8_W7.62mm_LongPads
- added C4: 0.1u, Capacitor_THT:C_Disc_D4.7mm_W2.5mm_P5.00mm, F.Cu at (124.5, 73.0)
- added G***: LOGO, project_parts:scanlines, B.Cu at (139.5, 63.0)
- added REF**: MountingHole_3.2mm_M3, MountingHole:MountingHole_3.2mm_M3, F.Cu at (186.6, 76.5)
- added REF**: MountingHole_3.2mm_M3, MountingHole:MountingHole_3.2mm_M3, F.Cu at (93.5, 76.5)
- added REF**: MountingHole_3.2mm_M3, MountingHole:MountingHole_3.2mm_M3, F.Cu at (186.5, 48.6)
- added REF**: MountingHole_3.2mm_M3, MountingHole:MountingHole_3.2mm_M3, F.Cu at (93.5, 48.5)
- R14: value 1.2k -> 1.5k
- R3: value 680 -> 1.2k
- R4: value 1.2 -> 1.2k
- R5: value 3.9k -> 4.7k
- R6: value 390 -> 680
- R7: value 2k -> 1.2k
- U1: value LM311 -> LM339; footprint Package_DIP:DIP-8_W7.62mm_LongPads -> Package_DIP:DIP-14_W7.62mm_LongPads
- moved R12 51.1 mm to (143.0, 62.9), turned to 180 degrees
- moved R13 32.4 mm to (124.4, 62.9)
- moved R6 24.2 mm to (153.9, 66.5)
- moved C1 10.1 mm to (96.1, 65.7), turned to 0 degrees
- moved U1 9.19 mm to (128.3, 77.9), turned to 90 degrees
- moved R1 7.52 mm to (121.0, 70.5)
- moved R4 7.52 mm to (100.5, 70.0)
- moved RV1 7.52 mm to (113.5, 78.5)
- moved C2 7.50 mm to (154.0, 72.5)
- moved R5 7.50 mm to (179.5, 70.0)
- moved R7 7.50 mm to (158.5, 70.0)
- moved RV2 7.50 mm to (171.5, 78.0)
- moved R3 5.90 mm to (146.3, 62.9)
- moved J2 5.10 mm to (181.2, 57.1)
- moved J1 4.60 mm to (98.9, 56.6)
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- renumbered U4 to U2
Connections:
- U1 pad 1: GND -> Net-(R6-Pad1)
- U1 pad 2: Net-(C3-Pad1) -> Net-(R3-Pad1)
- U1 pad 3: Net-(C1-Pad2) -> +5V
- U1 pad 4: GND -> Net-(C1-Pad2)
- U1 pad 5: Net-(U1-Pad5) -> Net-(C3-Pad1)
- U1 pad 6: Net-(U1-Pad6) -> Net-(C2-Pad2)
- U1 pad 7: Net-(R3-Pad1) -> Net-(C3-Pad1)
- U1 pad 8: +5V -> Net-(U1-Pad8)
Routing:
- net Net-(C3-Pad1): track 117.5 -> 51.1 mm
- net Net-(Q1-Pad2): track 101.8 -> 62.2 mm
- net +5V: track 159.6 -> 120.4 mm
- net Net-(R6-Pad1): track 13.2 -> 42.5 mm
- net +1.25V: track 50.8 -> 26.3 mm
- net Net-(R3-Pad1): track 10.1 -> 28.3 mm
- net Net-(C1-Pad2): track 32.2 -> 44.6 mm
- net Net-(R12-Pad1): track 28.5 -> 35.4 mm
- net Net-(C2-Pad2): track 36.2 -> 30.4 mm
- net Net-(J2-Pad1): track 11.4 -> 16.6 mm
- net Net-(C3-Pad2): track 25.8 -> 30.4 mm
- net Net-(R13-Pad1): track 12.1 -> 10.0 mm
Other:
- board text added: "levels"
- board text added: "two_comparator_effect 0.2 by Rob Schafer pcb by cyberboy666"
- board text removed: "2comparatorFX 0.1 by Rob Schafer pcb by cyberboy666"
- board text removed: "GREY"
- board text removed: "WHITE"

Commit message: update circuits
Parts:
- Q1, U2: footprint Package_TO_SOT_THT:TO-92_Inline -> Package_TO_SOT_THT:TO-92_HandSolder
Routing:
- net Net-(Q1-Pad2): track 62.2 -> 61.0 mm
- net +5V: track 120.4 -> 121.0 mm
Other:
- board text added: "two_comparator_effect by Rob Schafer pcb by cyberboy666 v0.2.1"
- board text removed: "two_comparator_effect 0.2 by Rob Schafer pcb by cyberboy666"
