File: two_comparator_effect/two_comparator_effect.kicad_pcb (KiCad board)
At the start: 2 copper layers, 100 x 35 mm, 34 parts, among them J1 RCA, J2 RCA, J3 Barrel_Jack, Q1 2N3904, U1 LM339, U2 LM317

Commit message: revised all boards
Parts:
- removed G***: LOGO, project_parts:scanlines
- J1, J2: value RCA -> rca; footprint lib_fp:RCJ-024 -> lib_fp:tht_rca_vertical
- moved C2 16.6 mm to (170.4, 70.0)
- moved R7 16.5 mm to (175.0, 70.0)
- moved R1 16.0 mm to (105.0, 70.1)
- moved RV1 10.2 mm to (123.7, 78.2)
- moved RV2 10.2 mm to (161.3, 78.1)
- moved C4 6.04 mm to (130.4, 71.7)
- moved U1 5.80 mm to (134.1, 77.9)
- moved R3 4.74 mm to (147.8, 58.4)
- moved R6 3.96 mm to (155.3, 62.8)
Routing:
- net Net-(R1-Pad2): track 7.66 -> 33.0 mm
- net Net-(R7-Pad2): track 8.16 -> 32.7 mm
- net Net-(R3-Pad1): track 28.3 -> 49.5 mm
- net +5V: track 121.0 -> 138.2 mm
- net Net-(R5-Pad2): track 8.16 -> 19.5 mm
- net Net-(R4-Pad2): track 8.36 -> 19.0 mm
- net Net-(R6-Pad1): track 42.5 -> 35.0 mm
- net Net-(C3-Pad1): track 51.1 -> 57.6 mm
- net Net-(R13-Pad1): track 10.0 -> 16.1 mm
- net Net-(R12-Pad1): track 35.4 -> 41.1 mm
- net Net-(C1-Pad2): track 44.6 -> 48.8 mm
- net Net-(C2-Pad2): track 30.4 -> 26.5 mm
- net Net-(Q1-Pad2): track 61.0 -> 60.3 mm
Other:
- board text added: "_^ 05"
- board text added: "two_comparator_effect v0_3 based on Rob Schafer design updated by cyberboy666"
- board text added: "underscores.shop"
- board text removed: "two_comparator_effect by Rob Schafer pcb by cyberboy666 v0.2.1"

Commit message: newest circuit revisions
Parts:
- added SW1: SW_DPDT_x2, lib:dpdt_mini_toggle_switch_tayda, F.Cu at (114.3, 41.6)
- RV1, RV2: value 1k -> 1k_pot
- moved U2 20.6 mm to (147.6, 51.2)
- moved R8 14.6 mm to (123.6, 46.8)
- moved R9 13.3 mm to (127.3, 46.8)
- moved R16 11.8 mm to (131.0, 46.8)
- moved R2 4.90 mm to (153.9, 47.0)
- moved R14 3.45 mm to (157.4, 47.0)
Connections:
- C3 pad 2: Net-(C3-Pad2) -> video_in
- J1 pad 1: Net-(C3-Pad2) -> Net-(J1-Pad1)
- R10 pad 1: Net-(J2-Pad1) -> video_out
- R8 pad 1: Net-(C3-Pad2) -> video_in
Routing:
- net video_out: track 0.00 -> 62.3 mm
- net Net-(J2-Pad1): track 16.6 -> 75.7 mm
- net Net-(C3-Pad2): track 30.4 -> 0.00 mm
- net Net-(J1-Pad1): track 0.00 -> 19.7 mm
- net video_in: track 0.00 -> 17.4 mm
- net +5V: track 138.2 -> 124.9 mm
- net +1.25V: track 26.3 -> 37.8 mm
- net Net-(SW1-Pad1): track 0.00 -> 4.70 mm
- net Net-(Q1-Pad2): track 60.3 -> 57.5 mm
Other:
- board text added: "two_comparator_effect v0_3_1 based on Rob Schafer design updated by cyberboy666"
- board text removed: "two_comparator_effect v0_3 based on Rob Schafer design updated by cyberboy666"

Commit message: updates
Parts:
- J1, J2: footprint lib_fp:tht_rca_vertical -> lib:tht_rca_vertical
- RV1, RV2: footprint lib_fp:Potentiometer_Vertical_Large -> lib:Potentiometer_Vertical_Large
