File: two_comparator_effect/two_comparator_effect.sch (KiCad schematic (older format))
At the start: 23 parts, among them J1 RCA, J2 RCA, Q1 2N3904, U1 LM311, U2 LM311, U3 LM317L_TO92

Commit message: routing boards
Parts:
- added C1: 1u, Capacitor_THT:C_Disc_D4.7mm_W2.5mm_P5.00mm, symbol Device:C
- added J3: Barrel_Jack, Connector_BarrelJack:BarrelJack_Horizontal, symbol Connector:Barrel_Jack_Switch
- added R1: 4.7k, Resistor_THT:R_Axial_DIN0207_L6.3mm_D2.5mm_P7.62mm_Horizontal, symbol Device:R
- added R3: 680, Resistor_THT:R_Axial_DIN0207_L6.3mm_D2.5mm_P7.62mm_Horizontal, symbol Device:R
- added R4: 1.2, Resistor_THT:R_Axial_DIN0207_L6.3mm_D2.5mm_P7.62mm_Horizontal, symbol Device:R
- added RV1: 1k, lib_fp:Potentiometer_Vertical_Large, symbol Device:R_POT
- added U1: LM311, Package_DIP:DIP-8_W7.62mm_LongPads, symbol Comparator:LM311
- C2: renamed from C1; footprint (none) -> Capacitor_THT:C_Disc_D4.7mm_W2.5mm_P5.00mm
- C3: renamed from C2; footprint (none) -> Capacitor_THT:C_Disc_D4.7mm_W2.5mm_P5.00mm
- D1: footprint (none) -> Diode_THT:D_A-405_P7.62mm_Horizontal
- J1, J2: footprint (none) -> lib_fp:RCJ-024
- R10: renamed from R7; footprint (none) -> Resistor_THT:R_Axial_DIN0207_L6.3mm_D2.5mm_P7.62mm_Horizontal
- R11: renamed from R8; footprint (none) -> Resistor_THT:R_Axial_DIN0207_L6.3mm_D2.5mm_P7.62mm_Horizontal
- R12: renamed from R9; footprint (none) -> Resistor_THT:R_Axial_DIN0207_L6.3mm_D2.5mm_P7.62mm_Horizontal
- R13: renamed from R10; footprint (none) -> Resistor_THT:R_Axial_DIN0207_L6.3mm_D2.5mm_P7.62mm_Horizontal
- R14: renamed from R11; footprint (none) -> Resistor_THT:R_Axial_DIN0207_L6.3mm_D2.5mm_P7.62mm_Horizontal
- R15: renamed from R12; footprint (none) -> Resistor_THT:R_Axial_DIN0207_L6.3mm_D2.5mm_P7.62mm_Horizontal
- R16: renamed from R13; footprint (none) -> Resistor_THT:R_Axial_DIN0207_L6.3mm_D2.5mm_P7.62mm_Horizontal
- R2: footprint (none) -> Resistor_THT:R_Axial_DIN0207_L6.3mm_D2.5mm_P7.62mm_Horizontal
- R5: renamed from R1; value 2.2k -> 3.9k; footprint (none) -> Resistor_THT:R_Axial_DIN0207_L6.3mm_D2.5mm_P7.62mm_Horizontal
- R6: renamed from R3; footprint (none) -> Resistor_THT:R_Axial_DIN0207_L6.3mm_D2.5mm_P7.62mm_Horizontal
- R7: renamed from R4; value 680 -> 2k; footprint (none) -> Resistor_THT:R_Axial_DIN0207_L6.3mm_D2.5mm_P7.62mm_Horizontal
- R8: renamed from R5; footprint (none) -> Resistor_THT:R_Axial_DIN0207_L6.3mm_D2.5mm_P7.62mm_Horizontal
- R9: renamed from R6; footprint (none) -> Resistor_THT:R_Axial_DIN0207_L6.3mm_D2.5mm_P7.62mm_Horizontal
- RV2: renamed from RV1; footprint (none) -> lib_fp:Potentiometer_Vertical_Large
- U2: renamed from U1; footprint (none) -> Package_DIP:DIP-8_W7.62mm_LongPads
- U3: renamed from U2; footprint (none) -> Package_DIP:DIP-8_W7.62mm_LongPads
- U4: renamed from U3; value LM317L_TO92 -> LM317; symbol Regulator_Linear:LM317L_TO92 -> Regulator_Linear:LM317_3PinPackage
Connections:
- wire segments 55 -> 77
- no-connect marks 4 -> 6
Other:
- note added: "POWER_SUPPLY"
- note added: "THRESHOLD_GREY"
- note added: "THRESHOLD_WHITE"
- note removed: "THRESHOLD"
- moved on the sheet: C2, C3, D1, J1, J2, Q1, R10, R11, R12, R13, R14, R15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

Commit message: updates to circuit
Parts:
- R3: value 680 -> 780
- R6: value 390 -> 780
Changed lines of the file:
@@
 P 6625 2850
 F 0 "R6" V 6418 2850 50  0000 C CNN
-F 1 "390" V 6509 2850 50  0000 C CNN
+F 1 "780" V 6509 2850 50  0000 C CNN
 F 2 "Resistor_THT:R_Axial_DIN0207_L6.3mm_D2.5mm_P7.62mm_Horizontal" V 6555 2850 50  0001 C CNN
 F 3 "~" H 6625 2850 50  0001 C CNN
@@
 P 6625 1550
 F 0 "R3" V 6418 1550 50  0000 C CNN
-F 1 "680" V 6509 1550 50  0000 C CNN
+F 1 "780" V 6509 1550 50  0000 C CNN
 F 2 "Resistor_THT:R_Axial_DIN0207_L6.3mm_D2.5mm_P7.62mm_Horizontal" V 6555 1550 50  0001 C CNN
 F 3 "~" H 6625 1550 50  0001 C CNN

Commit message: updated two_comparator and added two_point_one
Parts:
- removed U1, U2, U3: LM311, Package_DIP:DIP-8_W7.62mm_LongPads, symbol Comparator:LM311
- added C4: 0.1u, Capacitor_THT:C_Disc_D4.7mm_W2.5mm_P5.00mm, symbol Device:C
- added U1: LM339, Package_DIP:DIP-14_W7.62mm_LongPads, symbol Comparator:LM339
- R14: value 1.2k -> 1.5k
- R3: value 780 -> 1.2k
- R4: value 1.2 -> 1.2k
- R5: value 3.9k -> 4.7k
- R6: value 780 -> 680
- R7: value 2k -> 1.2k
- renumbered U4 to U2
Connections:
- net +5V: now also C4.1, U1.3 (V+)
- net GND: now also C4.2, U1.12 (V-)
- net at C3.1, D1.1 (K), R9.1: now also U1.11 (+), U1.5 (+), U1.7 (+)
- net at C2.2, RV2.2: now also U1.6 (-)
- net at R6.1: now also U1.1
- net at R12.1, R15.2: now also U1.10 (-)
- net at R13.1: now also U1.13
- net at C1.2, RV1.2: now also U1.4 (-)
- net at R3.1: now also U1.2
- no-connect marks 6 -> 3
Other:
- note added: "THRESHOLD_1"
- note added: "THRESHOLD_2"
- note removed: "THRESHOLD_GREY"
- note removed: "THRESHOLD_WHITE"
Changed lines of the file:
@@
 $EndDescr
 $Comp
-L Regulator_Linear:LM317_3PinPackage U4
+L Regulator_Linear:LM317_3PinPackage U2
 U 1 1 5EB5729E
 P 2200 5750
-F 0 "U4" H 2200 5992 50  0000 C CNN
+F 0 "U2" H 2200 5992 50  0000 C CNN
 F 1 "LM317" H 2200 5901 50  0000 C CNN
 F 2 "Package_TO_SOT_THT:TO-92_Inline" H 2200 5975 50  0001 C CIN
@@
 	3675 4050 3675 4150
 $Comp
-L power:+5V #PWR08
-U 1 1 5EB6363C
-P 5525 2425
-F 0 "#PWR08" H 5525 2275 50  0001 C CNN
-F 1 "+5V" H 5540 2598 50  0000 C CNN
-F 2 "" H 5525 2425 50  0001 C CNN
-F 3 "" H 5525 2425 50  0001 C CNN
-	1    5525 2425
-	1    0    0    -1
-$EndComp
-$Comp
-L power:GND #PWR09
-U 1 1 5EB65A5A
-P 5625 3225
-F 0 "#PWR09" H 5625 2975 50  0001 C CNN
-F 1 "GND" H 5630 3052 50  0000 C CNN
-F 2 "" H 5625 3225 50  0001 C CNN
-F 3 "" H 5625 3225 50  0001 C CNN
-	1    5625 3225
-	1    0    0    -1
-$EndComp
-Wire Wire Line
-	5525 3150 5525 3225
-Wire Wire Line
-	5525 3225 5625 3225
-Wire Wire Line
-	5625 3150 5625 3225
-Connection ~ 5625 3225
-Wire Wire Line
-	5525 2425 5525 2550
-NoConn ~ 5625 2550
-NoConn ~ 5725 2550
-$Comp
-L Comparator:LM311 U3
-U 1 1 5EB6703F
-P 5650 5275
-F 0 "U3" H 5994 5321 50  0000 L CNN
-F 1 "LM311" H 5994 5230 50  0000 L CNN
-F 2 "Package_DIP:DIP-8_W7.62mm_LongPads" H 5650 5275 50  0001 C CNN
-F 3 "http://www.ti.com/lit/ds/symlink/lm311.pdf" H 5650 5275 50  0001 C CNN
-	1    5650 5275
-	1    0    0    -1
-$EndComp
-$Comp
-L power:+5V #PWR018
-U 1 1 5EB67049
-P 5550 4850
-F 0 "#PWR018" H 5550 4700 50  0001 C CNN
-F 1 "+5V" H 5565 5023 50  0000 C CNN
-F 2 "" H 5550 4850 50  0001 C CNN
-F 3 "" H 5550 4850 50  0001 C CNN
-	1    5550 4850
-	1    0    0    -1
-$EndComp
-$Comp
-L power:GND #PWR020
-U 1 1 5EB67053
-P 5650 5650
-F 0 "#PWR020" H 5650 5400 50  0001 C CNN
-F 1 "GND" H 5655 5477 50  0000 C CNN
-F 2 "" H 5650 5650 50  0001 C CNN
-F 3 "" H 5650 5650 50  0001 C CNN
-	1    5650 5650
-	1    0    0    -1
-$EndComp
-Wire Wire Line
-	5550 5575 5550 5650
-Wire Wire Line
-	5550 5650 5650 5650
-Wire Wire Line
-	5650 5575 5650 5650
-Connection ~ 5650 5650
-Wire Wire Line
-	5550 4850 5550 4975
-NoConn ~ 5650 4975
-NoConn ~ 5750 4975
-$Comp
 L Device:C C2
 U 1 1 5EB6F7E6
@@
 P 4300 2600
 F 0 "R5" H 4370 2646 50  0000 L CNN
-F 1 "3.9k" H 4370 2555 50  0000 L CNN
+F 1 "4.7k" H 4370 2555 50  0000 L CNN
 F 2 "Resistor_THT:R_Axial_DIN0207_L6.3mm_D2.5mm_P7.62mm_Horizontal" V 4230 2600 50  0001 C CNN
 F 3 "~" H 4300 2600 50  0001 C CNN
@@
 P 4300 3300
 F 0 "R7" H 4231 3254 50  0000 R CNN
-F 1 "2k" H 4231 3345 50  0000 R CNN
+F 1 "1.2k" H 4231 3345 50  0000 R CNN
 F 2 "Resistor_THT:R_Axial_DIN0207_L6.3mm_D2.5mm_P7.62mm_Horizontal" V 4230 3300 50  0001 C CNN
 F 3 "~" H 4300 3300 50  0001 C CNN
@@
 Wire Wire Line
 	3675 4050 5075 4050
-$Comp
-L Comparator:LM311 U2
-U 1 1 5EB62130
-P 5625 2850
-F 0 "U2" H 5969 2896 50  0000 L CNN
-F 1 "LM311" H 5969 2805 50  0000 L CNN
-F 2 "Package_DIP:DIP-8_W7.62mm_LongPads" H 5625 2850 50  0001 C CNN
-F 3 "http://www.ti.com/lit/ds/symlink/lm311.pdf" H 5625 2850 50  0001 C CNN
-	1    5625 2850
-	1    0    0    -1
-$EndComp
 Wire Wire Line
 	5075 2750 5325 2750
@@
 P 6625 2850
 F 0 "R6" V 6418 2850 50  0000 C CNN
-F 1 "780" V 6509 2850 50  0000 C CNN
+F 1 "680" V 6509 2850 50  0000 C CNN
 F 2 "Resistor_THT:R_Axial_DIN0207_L6.3mm_D2.5mm_P7.62mm_Horizontal" V 6555 2850 50  0001 C CNN
 F 3 "~" H 6625 2850 50  0001 C CNN
@@
 P 7425 5475
 F 0 "R14" H 7355 5521 50  0000 R CNN
-F 1 "1.2k" H 7355 5430 50  0000 R CNN
+F 1 "1.5k" H 7355 5430 50  0000 R CNN
 F 2 "Resistor_THT:R_Axial_DIN0207_L6.3mm_D2.5mm_P7.62mm_Horizontal" V 7355 5475 50  0001 C CNN
 F 3 "~" H 7425 5475 50  0001 C CNN
@@
 BLACK & WHITE \nVIDEO OUT
 Text Notes 3600 2775 0    50   ~ 0
-THRESHOLD_WHITE
-$Comp
-L power:+5V #PWR03
-U 1 1 5EE7797F
-P 5525 1125
-F 0 "#PWR03" H 5525 975 50  0001 C CNN
-F 1 "+5V" H 5540 1298 50  0000 C CNN
-F 2 "" H 5525 1125 50  0001 C CNN
-F 3 "" H 5525 1125 50  0001 C CNN
-	1    5525 1125
-	1    0    0    -1
-$EndComp
-$Comp
-L power:GND #PWR04
-U 1 1 5EE77989
-P 5625 1925
-F 0 "#PWR04" H 5625 1675 50  0001 C CNN
-F 1 "GND" H 5630 1752 50  0000 C CNN
-F 2 "" H 5625 1925 50  0001 C CNN
-F 3 "" H 5625 1925 50  0001 C CNN
-	1    5625 1925
-	1    0    0    -1
-$EndComp
-Wire Wire Line
-	5525 1850 5525 1925
-Wire Wire Line
-	5525 1925 5625 1925
-Wire Wire Line
-	5625 1850 5625 1925
-Connection ~ 5625 1925
-Wire Wire Line
-	5525 1125 5525 1250
-NoConn ~ 5625 1250
-NoConn ~ 5725 1250
+THRESHOLD_2
 $Comp
 L Device:C C1
@@
 P 3500 2000
 F 0 "R4" H 3431 1954 50  0000 R CNN
-F 1 "1.2" H 3431 2045 50  0000 R CNN
+F 1 "1.2k" H 3431 2045 50  0000 R CNN
 F 2 "Resistor_THT:R_Axial_DIN0207_L6.3mm_D2.5mm_P7.62mm_Horizontal" V 3430 2000 50  0001 C CNN
 F 3 "~" H 3500 2000 50  0001 C CNN
@@
 Wire Wire Line
 	3650 1650 3875 1650
-$Comp
-L Comparator:LM311 U1
-U 1 1 5EE779E5
-P 5625 1550
-F 0 "U1" H 5969 1596 50  0000 L CNN
-F 1 "LM311" H 5969 1505 50  0000 L CNN
-F 2 "Package_DIP:DIP-8_W7.62mm_LongPads" H 5625 1550 50  0001 C CNN
-F 3 "http://www.ti.com/lit/ds/symlink/lm311.pdf" H 5625 1550 50  0001 C CNN
-	1    5625 1550
-	1    0    0    -1
-$EndComp
 Wire Wire Line
 	5075 1450 5325 1450
@@
 P 6625 1550
 F 0 "R3" V 6418 1550 50  0000 C CNN
-F 1 "780" V 6509 1550 50  0000 C CNN
+F 1 "1.2k" V 6509 1550 50  0000 C CNN
 F 2 "Resistor_THT:R_Axial_DIN0207_L6.3mm_D2.5mm_P7.62mm_Horizontal" V 6555 1550 50  0001 C CNN
 F 3 "~" H 6625 1550 50  0001 C CNN
@@
 	7425 1175 7425 1100
 Text Notes 2800 1500 0    50   ~ 0
-THRESHOLD_GREY
+THRESHOLD_1
 Connection ~ 5075 2750
 Wire Wire Line
@@
 Text Notes 1725 5325 0    50   ~ 0
 POWER_SUPPLY
+$Comp
+L Comparator:LM339 U1
+U 1 1 5F34098F
+P 5625 1550
+F 0 "U1" H 5625 1917 50  0000 C CNN
+F 1 "LM339" H 5625 1826 50  0000 C CNN
+F 2 "Package_DIP:DIP-14_W7.62mm_LongPads" H 5575 1650 50  0001 C CNN
+F 3 "http://www.ti.com/lit/ds/symlink/lm339.pdf" H 5675 1750 50  0001 C CNN
+	1    5625 1550
+	1    0    0    -1
+$EndComp
+$Comp
+L Comparator:LM339 U1
+U 2 1 5F34C782
+P 5625 2850
+F 0 "U1" H 5625 3217 50  0000 C CNN
+F 1 "LM339" H 5625 3126 50  0000 C CNN
+F 2 "Package_DIP:DIP-14_W7.62mm_LongPads" H 5575 2950 50  0001 C CNN
+F 3 "http://www.ti.com/lit/ds/symlink/lm339.pdf" H 5675 3050 50  0001 C CNN
+	2    5625 2850
+	1    0    0    -1
+$EndComp
+$Comp
+L Comparator:LM339 U1
+U 3 1 5F34D944
+P 5650 5275
+F 0 "U1" H 5650 5642 50  0000 C CNN
+F 1 "LM339" H 5650 5551 50  0000 C CNN
+F 2 "Package_DIP:DIP-14_W7.62mm_LongPads" H 5600 5375 50  0001 C CNN
+F 3 "http://www.ti.com/lit/ds/symlink/lm339.pdf" H 5700 5475 50  0001 C CNN
+	3    5650 5275
+	1    0    0    -1
+$EndComp
+$Comp
+L Comparator:LM339 U1
+U 4 1 5F350511
+P 6200 7175
+F 0 "U1" H 6200 7542 50  0000 C CNN
+F 1 "LM339" H 6200 7451 50  0000 C CNN
+F 2 "Package_DIP:DIP-14_W7.62mm_LongPads" H 6150 7275 50  0001 C CNN
+F 3 "http://www.ti.com/lit/ds/symlink/lm339.pdf" H 6250 7375 50  0001 C CNN
+	4    6200 7175
+	1    0    0    -1
+$EndComp
+$Comp
+L Comparator:LM339 U1
+U 5 1 5F3519B7
+P 5325 7150
+F 0 "U1" H 5283 7196 50  0000 L CNN
+F 1 "LM339" H 5283 7105 50  0000 L CNN
+F 2 "Package_DIP:DIP-14_W7.62mm_LongPads" H 5275 7250 50  0001 C CNN
+F 3 "http://www.ti.com/lit/ds/symlink/lm339.pdf" H 5375 7350 50  0001 C CNN
+	5    5325 7150
+	1    0    0    -1
+$EndComp
+NoConn ~ 5900 7075
+NoConn ~ 5900 7275
+NoConn ~ 6500 7175
+$Comp
+L power:+5V #PWR03
+U 1 1 5F355F1F
+P 5225 6850
+F 0 "#PWR03" H 5225 6700 50  0001 C CNN
+F 1 "+5V" H 5240 7023 50  0000 C CNN
+F 2 "" H 5225 6850 50  0001 C CNN
+F 3 "" H 5225 6850 50  0001 C CNN
+	1    5225 6850
+	1    0    0    -1
+$EndComp
+$Comp
+L power:GND #PWR04
+U 1 1 5F3567DE
+P 5225 7450
+F 0 "#PWR04" H 5225 7200 50  0001 C CNN
+F 1 "GND" H 5230 7277 50  0000 C CNN
+F 2 "" H 5225 7450 50  0001 C CNN
+F 3 "" H 5225 7450 50  0001 C CNN
+	1    5225 7450
+	1    0    0    -1
+$EndComp
+$Comp
+L Device:C C4
+U 1 1 5F35840A
+P 4875 7175
+F 0 "C4" H 4650 7250 50  0000 C CNN
+F 1 "0.1u" H 4650 7150 50  0000 C CNN
+F 2 "Capacitor_THT:C_Disc_D4.7mm_W2.5mm_P5.00mm" H 4913 7025 50  0001 C CNN
+F 3 "~" H 4875 7175 50  0001 C CNN
+	1    4875 7175
+	1    0    0    -1
+$EndComp
+Wire Wire Line
+	5225 6850 4875 6850
+Wire Wire Line
+	4875 6850 4875 7025
+Connection ~ 5225 6850
+$Comp
+L power:GND #PWR08
+U 1 1 5F35BEFF
+P 4875 7450
+F 0 "#PWR08" H 4875 7200 50  0001 C CNN
+F 1 "GND" H 4880 7277 50  0000 C CNN
+F 2 "" H 4875 7450 50  0001 C CNN
+F 3 "" H 4875 7450 50  0001 C CNN
+	1    4875 7450
+	1    0    0    -1
+$EndComp
+Wire Wire Line
+	4875 7325 4875 7450
 $EndSCHEMATC

Commit message: update circuits
Parts:
- Q1, U2: footprint Package_TO_SOT_THT:TO-92_Inline -> Package_TO_SOT_THT:TO-92_HandSolder
Changed lines of the file:
@@
 F 0 "U2" H 2200 5992 50  0000 C CNN
 F 1 "LM317" H 2200 5901 50  0000 C CNN
-F 2 "Package_TO_SOT_THT:TO-92_Inline" H 2200 5975 50  0001 C CIN
+F 2 "Package_TO_SOT_THT:TO-92_HandSolder" H 2200 5975 50  0001 C CIN
 F 3 "http://www.ti.com/lit/ds/snvs775k/snvs775k.pdf" H 2200 5750 50  0001 C CNN
 	1    2200 5750
@@
 F 0 "Q1" H 7815 4146 50  0000 L CNN
 F 1 "2N3904" H 7815 4055 50  0000 L CNN
-F 2 "Package_TO_SOT_THT:TO-92_Inline" H 7825 4025 50  0001 L CIN
+F 2 "Package_TO_SOT_THT:TO-92_HandSolder" H 7825 4025 50  0001 L CIN
 F 3 "https://www.fairchildsemi.com/datasheets/2N/2N3904.pdf" H 7625 4100 50  0001 L CNN
 	1    7625 4100
