File: chroma_luma_invert/blanking_and_burst.sch (KiCad schematic (older format))
At the start: 19 parts, among them U4 74HC4538, U5 74HC4538, U6 LM1881

Commit message: newest circuit revisions
Parts:
- C11: renamed from C12; value 0.001u -> 1n
- C13: renamed from C14; value 0.001u -> 1n
- R11: renamed from R16; value 12k -> 18k
- R14: renamed from R19; value 68k -> 75k
- renumbered C11 to C10, C13 to C12, C9 to C8, C10 to C9, R15 to R10, R17 to R12, R18 to R13, R14 to R9, RV4 to RV1, RV5 to RV2, RV6 to RV3, RV7 to RV4
Changed lines of the file:
@@
 blanking
 $Comp
-L power:+5V #PWR038
+L power:+5V #PWR035
 U 1 1 5EE76A17
 P 6400 1100
-F 0 "#PWR038" H 6400 950 50  0001 C CNN
+F 0 "#PWR035" H 6400 950 50  0001 C CNN
 F 1 "+5V" H 6415 1273 50  0000 C CNN
 F 2 "" H 6400 1100 50  0001 C CNN
@@
 $EndComp
 $Comp
-L Device:R R17
+L Device:R R12
 U 1 1 5EE76A1D
 P 6750 1500
-F 0 "R17" H 6680 1454 50  0000 R CNN
+F 0 "R12" H 6680 1454 50  0000 R CNN
 F 1 "10k" H 6680 1545 50  0000 R CNN
 F 2 "Resistor_THT:R_Axial_DIN0207_L6.3mm_D2.5mm_P7.62mm_Horizontal" V 6680 1500 50  0001 C CNN
@@
 $EndComp
 $Comp
-L Device:R_POT RV5
+L Device:R_POT RV2
 U 1 1 5EE76A23
 P 6400 1250
-F 0 "RV5" V 6193 1250 50  0000 C CNN
+F 0 "RV2" V 6193 1250 50  0000 C CNN
 F 1 "5k_trim" V 6284 1250 50  0000 C CNN
 F 2 "lib_fp:tht_vertical_trimpot_3362" H 6400 1250 50  0001 C CNN
@@
 $EndComp
 $Comp
-L Device:C_Small C12
+L Device:C_Small C11
 U 1 1 5EE76A29
 P 6850 1700
-F 0 "C12" V 6750 1500 50  0000 R CNN
-F 1 "0.001u" V 6850 1550 50  0000 R CNN
+F 0 "C11" V 6750 1500 50  0000 R CNN
+F 1 "1n" V 6850 1550 50  0000 R CNN
 F 2 "Capacitor_THT:C_Disc_D4.7mm_W2.5mm_P5.00mm" H 6888 1550 50  0001 C CNN
 F 3 "~" H 6850 1700 50  0001 C CNN
@@
 $EndComp
 $Comp
-L power:GND #PWR036
+L power:GND #PWR033
 U 1 1 5EE76A8D
 P 6200 2350
-F 0 "#PWR036" H 6200 2100 50  0001 C CNN
+F 0 "#PWR033" H 6200 2100 50  0001 C CNN
 F 1 "GND" H 6205 2177 50  0000 C CNN
 F 2 "" H 6200 2350 50  0001 C CNN
@@
 $EndComp
 $Comp
-L power:+5V #PWR043
+L power:+5V #PWR040
 U 1 1 5EE76A9A
 P 7900 1050
-F 0 "#PWR043" H 7900 900 50  0001 C CNN
+F 0 "#PWR040" H 7900 900 50  0001 C CNN
 F 1 "+5V" H 7915 1223 50  0000 C CNN
 F 2 "" H 7900 1050 50  0001 C CNN
@@
 $EndComp
 $Comp
-L Device:R R19
+L Device:R R14
 U 1 1 5EE76AA0
 P 8200 1450
-F 0 "R19" H 8130 1404 50  0000 R CNN
-F 1 "68k" H 8130 1495 50  0000 R CNN
+F 0 "R14" H 8130 1404 50  0000 R CNN
+F 1 "75k" H 8130 1495 50  0000 R CNN
 F 2 "Resistor_THT:R_Axial_DIN0207_L6.3mm_D2.5mm_P7.62mm_Horizontal" V 8130 1450 50  0001 C CNN
 F 3 "~" H 8200 1450 50  0001 C CNN
@@
 $EndComp
 $Comp
-L Device:R_POT RV7
+L Device:R_POT RV4
 U 1 1 5EE76AA6
 P 7900 1200
-F 0 "RV7" V 7693 1200 50  0000 C CNN
+F 0 "RV4" V 7693 1200 50  0000 C CNN
 F 1 "10k_trim" V 7784 1200 50  0000 C CNN
 F 2 "lib_fp:tht_vertical_trimpot_3362" H 7900 1200 50  0001 C CNN
@@
 $EndComp
 $Comp
-L Device:C_Small C14
+L Device:C_Small C13
 U 1 1 5EE76AAC
 P 8300 1700
-F 0 "C14" V 8200 1500 50  0000 R CNN
-F 1 "0.001u" V 8275 1575 50  0000 R CNN
+F 0 "C13" V 8200 1500 50  0000 R CNN
+F 1 "1n" V 8275 1575 50  0000 R CNN
 F 2 "Capacitor_THT:C_Disc_D4.7mm_W2.5mm_P5.00mm" H 8338 1550 50  0001 C CNN
 F 3 "~" H 8300 1700 50  0001 C CNN
@@
 $EndComp
 $Comp
-L power:GND #PWR041
+L power:GND #PWR038
 U 1 1 5EE76AC0
 P 7650 2700
-F 0 "#PWR041" H 7650 2450 50  0001 C CNN
+F 0 "#PWR038" H 7650 2450 50  0001 C CNN
 F 1 "GND" H 7655 2527 50  0000 C CNN
 F 2 "" H 7650 2700 50  0001 C CNN
@@
 NoConn ~ 8800 2400
 $Comp
-L power:+5V #PWR029
+L power:+5V #PWR026
 U 1 1 5EE76AD0
 P 2100 2550
-F 0 "#PWR029" H 2100 2400 50  0001 C CNN
+F 0 "#PWR026" H 2100 2400 50  0001 C CNN
 F 1 "+5V" H 2100 2700 50  0000 C CNN
 F 2 "" H 2100 2550 50  0001 C CNN
@@
 blanking_enable
 $Comp
-L Device:R R15
+L Device:R R10
 U 1 1 5ED36E19
 P 2100 2750
-F 0 "R15" H 2030 2704 50  0000 R CNN
+F 0 "R10" H 2030 2704 50  0000 R CNN
 F 1 "10k" H 2030 2795 50  0000 R CNN
 F 2 "Resistor_THT:R_Axial_DIN0207_L6.3mm_D2.5mm_P7.62mm_Horizontal" V 2030 2750 50  0001 C CNN
@@
 $EndComp
 $Comp
-L power:+5V #PWR037
+L power:+5V #PWR034
 U 1 1 5EEDDCB7
 P 6300 3850
-F 0 "#PWR037" H 6300 3700 50  0001 C CNN
+F 0 "#PWR034" H 6300 3700 50  0001 C CNN
 F 1 "+5V" H 6315 4023 50  0000 C CNN
 F 2 "" H 6300 3850 50  0001 C CNN
@@
 $EndComp
 $Comp
-L Device:R_POT RV4
+L Device:R_POT RV1
 U 1 1 5EEDDCC3
 P 6300 4000
-F 0 "RV4" V 6093 4000 50  0000 C CNN
+F 0 "RV1" V 6093 4000 50  0000 C CNN
 F 1 "10k_trim" V 6184 4000 50  0000 C CNN
 F 2 "lib_fp:tht_vertical_trimpot_3362" H 6300 4000 50  0001 C CNN
@@
 $EndComp
 $Comp
-L power:+5V #PWR042
+L power:+5V #PWR039
 U 1 1 5EEDDCD6
 P 7750 3850
-F 0 "#PWR042" H 7750 3700 50  0001 C CNN
+F 0 "#PWR039" H 7750 3700 50  0001 C CNN
 F 1 "+5V" H 7765 4023 50  0000 C CNN
 F 2 "" H 7750 3850 50  0001 C CNN
@@
 $EndComp
 $Comp
-L Device:R R18
+L Device:R R13
 U 1 1 5EEDDCDC
 P 8100 4250
-F 0 "R18" H 8030 4204 50  0000 R CNN
+F 0 "R13" H 8030 4204 50  0000 R CNN
 F 1 "22k" H 8030 4295 50  0000 R CNN
 F 2 "Resistor_THT:R_Axial_DIN0207_L6.3mm_D2.5mm_P7.62mm_Horizontal" V 8030 4250 50  0001 C CNN
@@
 $EndComp
 $Comp
-L Device:R_POT RV6
+L Device:R_POT RV3
 U 1 1 5EEDDCE2
 P 7750 4000
-F 0 "RV6" V 7543 4000 50  0000 C CNN
+F 0 "RV3" V 7543 4000 50  0000 C CNN
 F 1 "10k_trim" V 7634 4000 50  0000 C CNN
 F 2 "lib_fp:tht_vertical_trimpot_3362" H 7750 4000 50  0001 C CNN
@@
 $EndComp
 $Comp
-L Device:C_Small C13
+L Device:C_Small C12
 U 1 1 5EEDDCE8
 P 8200 4450
-F 0 "C13" V 8125 4275 50  0000 R CNN
+F 0 "C12" V 8125 4275 50  0000 R CNN
 F 1 "1uf" V 8200 4250 50  0000 R CNN
 F 2 "Capacitor_THT:C_Disc_D4.7mm_W2.5mm_P5.00mm" H 8238 4300 50  0001 C CNN
@@
 v_blanking
 $Comp
-L power:+5V #PWR039
+L power:+5V #PWR036
 U 1 1 5EF1C3EF
 P 7500 4850
-F 0 "#PWR039" H 7500 4700 50  0001 C CNN
+F 0 "#PWR036" H 7500 4700 50  0001 C CNN
 F 1 "+5V" H 7500 5000 50  0000 C CNN
 F 2 "" H 7500 4850 50  0001 C CNN
@@
 $EndComp
 $Comp
-L power:+5V #PWR026
+L power:+5V #PWR023
 U 1 1 5EFF6827
 P 1250 6325
-F 0 "#PWR026" H 1250 6175 50  0001 C CNN
+F 0 "#PWR023" H 1250 6175 50  0001 C CNN
 F 1 "+5V" H 1265 6498 50  0000 C CNN
 F 2 "" H 1250 6325 50  0001 C CNN
@@
 $EndComp
 $Comp
-L power:GND #PWR027
+L power:GND #PWR024
 U 1 1 5EFF716E
 P 1250 7325
-F 0 "#PWR027" H 1250 7075 50  0001 C CNN
+F 0 "#PWR024" H 1250 7075 50  0001 C CNN
 F 1 "GND" H 1255 7152 50  0000 C CNN
 F 2 "" H 1250 7325 50  0001 C CNN
@@
 $EndComp
 $Comp
-L power:+5V #PWR030
+L power:+5V #PWR027
 U 1 1 5EFF9529
 P 2150 6325
-F 0 "#PWR030" H 2150 6175 50  0001 C CNN
+F 0 "#PWR027" H 2150 6175 50  0001 C CNN
 F 1 "+5V" H 2165 6498 50  0000 C CNN
 F 2 "" H 2150 6325 50  0001 C CNN
@@
 $EndComp
 $Comp
-L power:GND #PWR031
+L power:GND #PWR028
 U 1 1 5EFF9533
 P 2150 7325
-F 0 "#PWR031" H 2150 7075 50  0001 C CNN
+F 0 "#PWR028" H 2150 7075 50  0001 C CNN
 F 1 "GND" H 2155 7152 50  0000 C CNN
 F 2 "" H 2150 7325 50  0001 C CNN
@@
 $EndComp
 $Comp
-L Device:C_Small C11
+L Device:C_Small C10
 U 1 1 5EEDDCC9
 P 6750 4450
-F 0 "C11" V 6650 4250 50  0000 R CNN
+F 0 "C10" V 6650 4250 50  0000 R CNN
 F 1 "0.1uf" V 6800 4250 50  0000 R CNN
 F 2 "Capacitor_THT:C_Disc_D4.7mm_W2.5mm_P5.00mm" H 6788 4300 50  0001 C CNN
@@
 $EndComp
 $Comp
-L Device:R R16
+L Device:R R11
 U 1 1 5EEDDCBD
 P 6650 4150
-F 0 "R16" H 6580 4104 50  0000 R CNN
-F 1 "12k" H 6580 4195 50  0000 R CNN
+F 0 "R11" H 6580 4104 50  0000 R CNN
+F 1 "18k" H 6580 4195 50  0000 R CNN
 F 2 "Resistor_THT:R_Axial_DIN0207_L6.3mm_D2.5mm_P7.62mm_Horizontal" V 6580 4150 50  0001 C CNN
 F 3 "~" H 6650 4150 50  0001 C CNN
@@
 $EndComp
 $Comp
-L power:+5V #PWR035
+L power:+5V #PWR032
 U 1 1 5EF0BEB6
 P 6050 4850
-F 0 "#PWR035" H 6050 4700 50  0001 C CNN
+F 0 "#PWR032" H 6050 4700 50  0001 C CNN
 F 1 "+5V" H 6050 5000 50  0000 C CNN
 F 2 "" H 6050 4850 50  0001 C CNN
@@
 	6050 5250 6250 5250
 $Comp
-L power:GND #PWR040
+L power:GND #PWR037
 U 1 1 5EEDDCF5
 P 7600 5400
-F 0 "#PWR040" H 7600 5150 50  0001 C CNN
+F 0 "#PWR037" H 7600 5150 50  0001 C CNN
 F 1 "GND" H 7600 5200 50  0000 C CNN
 F 2 "" H 7600 5400 50  0001 C CNN
@@
 $EndComp
 $Comp
-L Device:C_Small C9
+L Device:C_Small C8
 U 1 1 61570AC5
 P 1850 3850
-F 0 "C9" V 1650 3900 50  0000 R CNN
+F 0 "C8" V 1650 3900 50  0000 R CNN
 F 1 "0.1u" V 1750 3950 50  0000 R CNN
 F 2 "Capacitor_THT:C_Disc_D4.7mm_W2.5mm_P5.00mm" H 1888 3700 50  0001 C CNN
@@
 $EndComp
 $Comp
-L Device:R R14
+L Device:R R9
 U 1 1 61575026
 P 1850 4150
-F 0 "R14" V 1950 4200 50  0000 R CNN
+F 0 "R9" V 1950 4200 50  0000 R CNN
 F 1 "680k" V 1850 4250 50  0000 R CNN
 F 2 "Resistor_THT:R_Axial_DIN0207_L6.3mm_D2.5mm_P7.62mm_Horizontal" V 1780 4150 50  0001 C CNN
@@
 $EndComp
 $Comp
-L Device:C_Small C10
+L Device:C_Small C9
 U 1 1 6157A6B8
 P 1850 4500
-F 0 "C10" V 1650 4600 50  0000 R CNN
+F 0 "C9" V 1650 4600 50  0000 R CNN
 F 1 "0.1u" V 1750 4600 50  0000 R CNN
 F 2 "Capacitor_THT:C_Disc_D4.7mm_W2.5mm_P5.00mm" H 1888 4350 50  0001 C CNN
@@
 	1750 3850 1600 3850
 $Comp
-L power:GND #PWR028
+L power:GND #PWR025
 U 1 1 6157C08B
 P 1550 4600
-F 0 "#PWR028" H 1550 4350 50  0001 C CNN
+F 0 "#PWR025" H 1550 4350 50  0001 C CNN
 F 1 "GND" H 1555 4427 50  0000 C CNN
 F 2 "" H 1550 4600 50  0001 C CNN
@@
 Connection ~ 3300 3950
 $Comp
-L power:+5V #PWR032
+L power:+5V #PWR029
 U 1 1 615A82DC
 P 2600 3550
-F 0 "#PWR032" H 2600 3400 50  0001 C CNN
+F 0 "#PWR029" H 2600 3400 50  0001 C CNN
 F 1 "+5V" H 2615 3723 50  0000 C CNN
 F 2 "" H 2600 3550 50  0001 C CNN
@@
 	6050 4850 6050 5250
 $Comp
-L power:GND #PWR033
+L power:GND #PWR030
 U 1 1 61605B1C
 P 2600 4250
-F 0 "#PWR033" H 2600 4000 50  0001 C CNN
+F 0 "#PWR030" H 2600 4000 50  0001 C CNN
 F 1 "GND" H 2605 4077 50  0000 C CNN
 F 2 "" H 2600 4250 50  0001 C CNN
@@
 $EndComp
 $Comp
-L power:GND #PWR034
+L power:GND #PWR031
 U 1 1 61605EFE
 P 5800 5300
-F 0 "#PWR034" H 5800 5050 50  0001 C CNN
+F 0 "#PWR031" H 5800 5050 50  0001 C CNN
 F 1 "GND" H 5805 5127 50  0000 C CNN
 F 2 "" H 5800 5300 50  0001 C CNN
