File: chroma_luma_invert/chroma_luma_invert.sch (KiCad schematic (older format))
At the start: 26 parts, among them U1 AD8042, U2 AD8042

Commit message: routing boards
Parts:
- added J3: Barrel_Jack, Connector_BarrelJack:BarrelJack_Horizontal, symbol Connector:Barrel_Jack_Switch
- added unit 3 of U1
- added unit 3 of U2
- C1: renamed from C?; footprint (none) -> Capacitor_THT:C_Disc_D4.7mm_W2.5mm_P5.00mm
- D1: renamed from D?; footprint (none) -> Diode_THT:D_DO-41_SOD81_P7.62mm_Horizontal
- J1, J2: renamed from J?; footprint (none) -> lib_fp:RCJ-024
- J4: renamed from J?; footprint (none) -> Connector_PinHeader_2.54mm:PinHeader_1x12_P2.54mm_Vertical
- R1, R10, R11, R12, R13, R14, R15, R2, R3, R4, R5, R6, R7, R8, R9: renamed from R?; footprint (none) -> Resistor_THT:R_Axial_DIN0207_L6.3mm_D2.5mm_P7.62mm_Horizontal
- SW1, SW2: renamed from SW?; footprint (none) -> lib_fp:mini_toggle_switch_tayda; symbol Switch:SW_SPST -> Switch:SW_SPDT
- U1, U2: footprint (none) -> Package_DIP:DIP-8_W7.62mm_LongPads
- U3: renamed from U?; footprint (none) -> Package_DIP:DIP-16_W7.62mm_LongPads
- U4: renamed from U?; value LM317L_TO92 -> LM317; footprint Package_TO_SOT_THT:TO-92_Inline -> Package_TO_SOT_THT:TO-220-3_Horizontal_TabDown; symbol Regulator_Linear:LM317L_TO92 -> Regulator_Linear:LM317_3PinPackage
Connections:
- wire segments 107 -> 111
- no-connect marks 6 -> 8

Commit message: updated opamp
Parts:
- removed unit 3 of U2
- U1: value AD8042 -> AD8044; footprint Package_DIP:DIP-8_W7.62mm_LongPads -> Package_DIP:DIP-14_W7.62mm_LongPads; symbol Amplifier_Operational:ADA4807-2ARM -> Amplifier_Operational:ADA4807-4
- U1: renamed from U2; value AD8042 -> AD8044; footprint Package_DIP:DIP-8_W7.62mm_LongPads -> Package_DIP:DIP-14_W7.62mm_LongPads; symbol Amplifier_Operational:ADA4807-2ARM -> Amplifier_Operational:ADA4807-4
Changed lines of the file:
@@
 	2425 1600 2425 1550
 $Comp
-L Amplifier_Operational:ADA4807-2ARM U1
+L Amplifier_Operational:ADA4807-4 U1
 U 1 1 5EBBB1FA
 P 3400 1650
 F 0 "U1" H 3400 2017 50  0000 C CNN
-F 1 "AD8042" H 3400 1926 50  0000 C CNN
-F 2 "Package_DIP:DIP-8_W7.62mm_LongPads" H 3400 1650 50  0001 C CNN
+F 1 "AD8044" H 3400 1926 50  0000 C CNN
+F 2 "Package_DIP:DIP-14_W7.62mm_LongPads" H 3400 1650 50  0001 C CNN
 F 3 "https://www.analog.com/media/en/technical-documentation/data-sheets/ADA4807-1_4807-2_4807-4.pdf" H 3400 1650 50  0001 C CNN
 	1    3400 1650
@@
 	3100 2450 3100 2600
 $Comp
-L Amplifier_Operational:ADA4807-2ARM U2
-U 2 1 5EBD1190
+L Amplifier_Operational:ADA4807-4 U1
+U 3 1 5EBD1190
 P 5600 3475
-F 0 "U2" H 5600 3108 50  0000 C CNN
-F 1 "AD8042" H 5600 3199 50  0000 C CNN
-F 2 "Package_DIP:DIP-8_W7.62mm_LongPads" H 5600 3475 50  0001 C CNN
+F 0 "U1" H 5600 3108 50  0000 C CNN
+F 1 "AD8044" H 5600 3199 50  0000 C CNN
+F 2 "Package_DIP:DIP-14_W7.62mm_LongPads" H 5600 3475 50  0001 C CNN
 F 3 "https://www.analog.com/media/en/technical-documentation/data-sheets/ADA4807-1_4807-2_4807-4.pdf" H 5600 3475 50  0001 C CNN
-	2    5600 3475
+	3    5600 3475
 	1    0    0    1
 $EndComp
@@
 $EndComp
 $Comp
-L Amplifier_Operational:ADA4807-2ARM U2
-U 1 1 5EBC7462
+L Amplifier_Operational:ADA4807-4 U1
+U 2 1 5EBC7462
 P 5625 1750
-F 0 "U2" H 5675 1500 50  0000 C CNN
-F 1 "AD8042" H 5675 1575 50  0000 C CNN
-F 2 "Package_DIP:DIP-8_W7.62mm_LongPads" H 5625 1750 50  0001 C CNN
+F 0 "U1" H 5675 1500 50  0000 C CNN
+F 1 "AD8044" H 5675 1575 50  0000 C CNN
+F 2 "Package_DIP:DIP-14_W7.62mm_LongPads" H 5625 1750 50  0001 C CNN
 F 3 "https://www.analog.com/media/en/technical-documentation/data-sheets/ADA4807-1_4807-2_4807-4.pdf" H 5625 1750 50  0001 C CNN
-	1    5625 1750
+	2    5625 1750
 	1    0    0    1
 $EndComp
@@
 switcher
 $Comp
-L Amplifier_Operational:ADA4807-2ARM U1
-U 2 1 5EC1C2E9
+L Amplifier_Operational:ADA4807-4 U1
+U 4 1 5EC1C2E9
 P 9375 1325
 F 0 "U1" H 9375 1692 50  0000 C CNN
-F 1 "AD8042" H 9375 1601 50  0000 C CNN
-F 2 "Package_DIP:DIP-8_W7.62mm_LongPads" H 9375 1325 50  0001 C CNN
+F 1 "AD8044" H 9375 1601 50  0000 C CNN
+F 2 "Package_DIP:DIP-14_W7.62mm_LongPads" H 9375 1325 50  0001 C CNN
 F 3 "https://www.analog.com/media/en/technical-documentation/data-sheets/ADA4807-1_4807-2_4807-4.pdf" H 9375 1325 50  0001 C CNN
-	2    9375 1325
+	4    9375 1325
 	1    0    0    -1
 $EndComp
@@
 	1375 4025 1375 4225
 $Comp
-L Amplifier_Operational:ADA4807-2ARM U1
-U 3 1 5EECCE6A
+L Amplifier_Operational:ADA4807-4 U1
+U 5 1 5EECCE6A
 P 1175 5325
 F 0 "U1" H 1175 5600 50  0000 C CNN
-F 1 "AD8042" H 1250 5525 50  0000 C CNN
-F 2 "Package_DIP:DIP-8_W7.62mm_LongPads" H 1175 5325 50  0001 C CNN
+F 1 "AD8044" H 1250 5525 50  0000 C CNN
+F 2 "Package_DIP:DIP-14_W7.62mm_LongPads" H 1175 5325 50  0001 C CNN
 F 3 "https://www.analog.com/media/en/technical-documentation/data-sheets/ADA4807-1_4807-2_4807-4.pdf" H 1175 5325 50  0001 C CNN
-	3    1175 5325
-	1    0    0    -1
-$EndComp
-$Comp
-L Amplifier_Operational:ADA4807-2ARM U2
-U 3 1 5EED0088
-P 1600 5325
-F 0 "U2" H 1325 5600 50  0000 C CNN
-F 1 "AD8042" H 1250 5525 50  0000 C CNN
-F 2 "Package_DIP:DIP-8_W7.62mm_LongPads" H 1600 5325 50  0001 C CNN
-F 3 "https://www.analog.com/media/en/technical-documentation/data-sheets/ADA4807-1_4807-2_4807-4.pdf" H 1600 5325 50  0001 C CNN
-	3    1600 5325
-	-1   0    0    -1
+	5    1175 5325
+	1    0    0    -1
 $EndComp
 $Comp
@@
 $EndComp
 $Comp
-L power:+5V #PWR0102
-U 1 1 5EED48FC
-P 1700 5025
-F 0 "#PWR0102" H 1700 4875 50  0001 C CNN
-F 1 "+5V" H 1715 5198 50  0000 C CNN
-F 2 "" H 1700 5025 50  0001 C CNN
-F 3 "" H 1700 5025 50  0001 C CNN
-	1    1700 5025
-	1    0    0    -1
-$EndComp
-$Comp
 L power:GND #PWR0103
 U 1 1 5EED4E41
@@
 	1    0    0    -1
 $EndComp
-$Comp
-L power:GND #PWR0104
-U 1 1 5EED534C
-P 1700 5625
-F 0 "#PWR0104" H 1700 5375 50  0001 C CNN
-F 1 "GND" H 1705 5452 50  0000 C CNN
-F 2 "" H 1700 5625 50  0001 C CNN
-F 3 "" H 1700 5625 50  0001 C CNN
-	1    1700 5625
-	1    0    0    -1
-$EndComp

Commit message: updated two_comparator and added two_point_one
Parts:
- added C10, C11, C12, C13, C14, C15, C9: 0.1u, Capacitor_THT:C_Disc_D4.7mm_W2.5mm_P5.00mm, symbol Device:C
- added C8: 10uf, Capacitor_THT:CP_Radial_D6.3mm_P2.50mm, symbol Device:CP1
- R8: value 2.2 -> 2.2k
Connections:
- net +5V: now also C10.2, C11.2, C12.2, C13.2, C14.2, C15.2, C8.1, C9.2; no longer U3.6 (Inh)
- net GND: now also U3.6 (Inh), C10.1, C11.1, C12.1, C13.1, C14.1, C15.1, C8.2, C9.1
Changed lines of the file:
@@
 U 1 1 5EBDE023
 P 8050 1825
-F 0 "U3" H 8594 1871 50  0000 L CNN
-F 1 "4051" H 8594 1780 50  0000 L CNN
+F 0 "U3" H 8200 2775 50  0000 L CNN
+F 1 "4051" H 8200 2675 50  0000 L CNN
 F 2 "Package_DIP:DIP-16_W7.62mm_LongPads" H 8050 1825 50  0001 C CNN
 F 3 "http://www.intersil.com/content/dam/Intersil/documents/cd40/cd4051bms-52bms-53bms.pdf" H 8050 1825 50  0001 C CNN
@@
 P 4750 1800
 F 0 "R8" H 4680 1754 50  0000 R CNN
-F 1 "2.2" H 4680 1845 50  0000 R CNN
+F 1 "2.2k" H 4680 1845 50  0000 R CNN
 F 2 "Resistor_THT:R_Axial_DIN0207_L6.3mm_D2.5mm_P7.62mm_Horizontal" V 4680 1800 50  0001 C CNN
 F 3 "~" H 4750 1800 50  0001 C CNN
@@
 	1    0    0    -1
 $EndComp
-$Comp
-L power:+5V #PWR07
-U 1 1 5EC0DF3A
-P 7325 2100
-F 0 "#PWR07" H 7325 1950 50  0001 C CNN
-F 1 "+5V" H 7340 2273 50  0000 C CNN
-F 2 "" H 7325 2100 50  0001 C CNN
-F 3 "" H 7325 2100 50  0001 C CNN
-	1    7325 2100
-	1    0    0    -1
-$EndComp
-Wire Wire Line
-	7550 2125 7325 2125
-Wire Wire Line
-	7325 2125 7325 2100
 Text Notes 4275 775  0    79   ~ 0
 original_video
@@
 NoConn ~ 3650 5500
 NoConn ~ 3650 5850
+Wire Wire Line
+	7550 2125 7500 2125
+Wire Wire Line
+	7500 2125 7500 2425
+Connection ~ 7500 2425
+$Comp
+L power:+5V #PWR07
+U 1 1 5F3A990E
+P 3775 6725
+F 0 "#PWR07" H 3775 6575 50  0001 C CNN
+F 1 "+5V" H 3790 6898 50  0000 C CNN
+F 2 "" H 3775 6725 50  0001 C CNN
+F 3 "" H 3775 6725 50  0001 C CNN
+	1    3775 6725
+	1    0    0    -1
+$EndComp
+$Comp
+L Device:C C9
+U 1 1 5F3AEB5B
+P 4150 6875
+F 0 "C9" H 3975 6775 50  0000 C CNN
+F 1 "0.1u" H 3950 6850 50  0000 C CNN
+F 2 "Capacitor_THT:C_Disc_D4.7mm_W2.5mm_P5.00mm" H 4188 6725 50  0001 C CNN
+F 3 "~" H 4150 6875 50  0001 C CNN
+	1    4150 6875
+	-1   0    0    1
+$EndComp
+$Comp
+L power:GND #PWR021
+U 1 1 5F3AF915
+P 4150 7025
+F 0 "#PWR021" H 4150 6775 50  0001 C CNN
+F 1 "GND" H 4155 6852 50  0000 C CNN
+F 2 "" H 4150 7025 50  0001 C CNN
+F 3 "" H 4150 7025 50  0001 C CNN
+	1    4150 7025
+	1    0    0    -1
+$EndComp
+$Comp
+L Device:C C10
+U 1 1 5F3AFD97
+P 4550 6875
+F 0 "C10" H 4375 6775 50  0000 C CNN
+F 1 "0.1u" H 4350 6850 50  0000 C CNN
+F 2 "Capacitor_THT:C_Disc_D4.7mm_W2.5mm_P5.00mm" H 4588 6725 50  0001 C CNN
+F 3 "~" H 4550 6875 50  0001 C CNN
+	1    4550 6875
+	-1   0    0    1
+$EndComp
+$Comp
+L Device:C C11
+U 1 1 5F3B0751
+P 4925 6875
+F 0 "C11" H 4750 6775 50  0000 C CNN
+F 1 "0.1u" H 4725 6850 50  0000 C CNN
+F 2 "Capacitor_THT:C_Disc_D4.7mm_W2.5mm_P5.00mm" H 4963 6725 50  0001 C CNN
+F 3 "~" H 4925 6875 50  0001 C CNN
+	1    4925 6875
+	-1   0    0    1
+$EndComp
+$Comp
+L Device:C C12
+U 1 1 5F3B0F11
+P 5325 6875
+F 0 "C12" H 5150 6775 50  0000 C CNN
+F 1 "0.1u" H 5125 6850 50  0000 C CNN
+F 2 "Capacitor_THT:C_Disc_D4.7mm_W2.5mm_P5.00mm" H 5363 6725 50  0001 C CNN
+F 3 "~" H 5325 6875 50  0001 C CNN
+	1    5325 6875
+	-1   0    0    1
+$EndComp
+$Comp
+L Device:C C13
+U 1 1 5F3B19F6
+P 5725 6875
+F 0 "C13" H 5550 6775 50  0000 C CNN
+F 1 "0.1u" H 5525 6850 50  0000 C CNN
+F 2 "Capacitor_THT:C_Disc_D4.7mm_W2.5mm_P5.00mm" H 5763 6725 50  0001 C CNN
+F 3 "~" H 5725 6875 50  0001 C CNN
+	1    5725 6875
+	-1   0    0    1
+$EndComp
+$Comp
+L Device:C C14
+U 1 1 5F3B2212
+P 6125 6875
+F 0 "C14" H 5950 6775 50  0000 C CNN
+F 1 "0.1u" H 5925 6850 50  0000 C CNN
+F 2 "Capacitor_THT:C_Disc_D4.7mm_W2.5mm_P5.00mm" H 6163 6725 50  0001 C CNN
+F 3 "~" H 6125 6875 50  0001 C CNN
+	1    6125 6875
+	-1   0    0    1
+$EndComp
+$Comp
+L Device:C C15
+U 1 1 5F3B2B2B
+P 6525 6875
+F 0 "C15" H 6350 6775 50  0000 C CNN
+F 1 "0.1u" H 6325 6850 50  0000 C CNN
+F 2 "Capacitor_THT:C_Disc_D4.7mm_W2.5mm_P5.00mm" H 6563 6725 50  0001 C CNN
+F 3 "~" H 6525 6875 50  0001 C CNN
+	1    6525 6875
+	-1   0    0    1
+$EndComp
+$Comp
+L power:GND #PWR023
+U 1 1 5F3B3278
+P 4550 7025
+F 0 "#PWR023" H 4550 6775 50  0001 C CNN
+F 1 "GND" H 4555 6852 50  0000 C CNN
+F 2 "" H 4550 7025 50  0001 C CNN
+F 3 "" H 4550 7025 50  0001 C CNN
+	1    4550 7025
+	1    0    0    -1
+$EndComp
+$Comp
+L power:GND #PWR024
+U 1 1 5F3B3611
+P 4925 7025
+F 0 "#PWR024" H 4925 6775 50  0001 C CNN
+F 1 "GND" H 4930 6852 50  0000 C CNN
+F 2 "" H 4925 7025 50  0001 C CNN
+F 3 "" H 4925 7025 50  0001 C CNN
+	1    4925 7025
+	1    0    0    -1
+$EndComp
+$Comp
+L power:GND #PWR037
+U 1 1 5F3B39DD
+P 5325 7025
+F 0 "#PWR037" H 5325 6775 50  0001 C CNN
+F 1 "GND" H 5330 6852 50  0000 C CNN
+F 2 "" H 5325 7025 50  0001 C CNN
+F 3 "" H 5325 7025 50  0001 C CNN
+	1    5325 7025
+	1    0    0    -1
+$EndComp
+$Comp
+L power:GND #PWR047
+U 1 1 5F3B3F41
+P 5725 7025
+F 0 "#PWR047" H 5725 6775 50  0001 C CNN
+F 1 "GND" H 5730 6852 50  0000 C CNN
+F 2 "" H 5725 7025 50  0001 C CNN
+F 3 "" H 5725 7025 50  0001 C CNN
+	1    5725 7025
+	1    0    0    -1
+$EndComp
+$Comp
+L power:GND #PWR048
+U 1 1 5F3B452D
+P 6125 7025
+F 0 "#PWR048" H 6125 6775 50  0001 C CNN
+F 1 "GND" H 6130 6852 50  0000 C CNN
+F 2 "" H 6125 7025 50  0001 C CNN
+F 3 "" H 6125 7025 50  0001 C CNN
+	1    6125 7025
+	1    0    0    -1
+$EndComp
+$Comp
+L power:GND #PWR049
+U 1 1 5F3B48D7
+P 6525 7025
+F 0 "#PWR049" H 6525 6775 50  0001 C CNN
+F 1 "GND" H 6530 6852 50  0000 C CNN
+F 2 "" H 6525 7025 50  0001 C CNN
+F 3 "" H 6525 7025 50  0001 C CNN
+	1    6525 7025
+	1    0    0    -1
+$EndComp
+$Comp
+L Device:CP1 C8
+U 1 1 5F3B5622
+P 3775 6875
+F 0 "C8" H 3900 6975 50  0000 L CNN
+F 1 "10uf" H 3900 6875 50  0000 L CNN
+F 2 "Capacitor_THT:CP_Radial_D6.3mm_P2.50mm" H 3775 6875 50  0001 C CNN
+F 3 "~" H 3775 6875 50  0001 C CNN
+	1    3775 6875
+	1    0    0    -1
+$EndComp
+$Comp
+L power:GND #PWR019
+U 1 1 5F3B6A73
+P 3775 7025
+F 0 "#PWR019" H 3775 6775 50  0001 C CNN
+F 1 "GND" H 3780 6852 50  0000 C CNN
+F 2 "" H 3775 7025 50  0001 C CNN
+F 3 "" H 3775 7025 50  0001 C CNN
+	1    3775 7025
+	1    0    0    -1
+$EndComp
+Wire Wire Line
+	3775 6725 4150 6725
+Connection ~ 3775 6725
+Connection ~ 4150 6725
+Wire Wire Line
+	4150 6725 4550 6725
+Connection ~ 4550 6725
+Wire Wire Line
+	4550 6725 4925 6725
+Connection ~ 4925 6725
+Wire Wire Line
+	4925 6725 5325 6725
+Connection ~ 5325 6725
+Wire Wire Line
+	5325 6725 5725 6725
+Connection ~ 5725 6725
+Wire Wire Line
+	5725 6725 6125 6725
+Connection ~ 6125 6725
+Wire Wire Line
+	6125 6725 6525 6725
 $EndSCHEMATC

Commit message: revised all boards
Parts:
- removed R1: 1.5k, Resistor_THT:R_Axial_DIN0207_L6.3mm_D2.5mm_P7.62mm_Horizontal, symbol Device:R
- removed R12: 1k, Resistor_THT:R_Axial_DIN0207_L6.3mm_D2.5mm_P7.62mm_Horizontal, symbol Device:R
- added C16: 0.001u, Capacitor_THT:C_Disc_D4.7mm_W2.5mm_P5.00mm, symbol Device:C
- added RV5, RV6, RV7: 1k_trim, lib_fp:tht_vertical_trimpot_3362, symbol Device:R_POT
- J1, J2: footprint lib_fp:RCJ-024 -> lib_fp:tht_vertical_rca
- R3: value 1k -> 1.5k
- SW1, SW2: value SW_SPST -> SPDT
- U1: footprint Package_DIP:DIP-14_W7.62mm_LongPads -> project_parts:DIP+SOIC_14
- U3: value 4051 -> CD4051
Connections:
- net GND: now also C16.2
- net invert_burst: now also RV6.2, RV7.1; no longer U3.15 (X2)
- net invert_video: now also RV5.2
- net at R3.2, R4.1, R8.2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: now also RV5.1
- net at R11.1, R13.1, U1.9 (-): now also RV6.1
- new net: C16.1, RV7.2, U3.15 (X2)
- no-connect marks 8 -> 11
Other:
- note added: "rc delay filter"
Changed lines of the file:
@@
 F 0 "J1" H 1203 1788 50  0000 C CNN
 F 1 "rca" H 1203 1697 50  0000 C CNN
-F 2 "lib_fp:RCJ-024" H 1275 1550 50  0001 C CNN
+F 2 "lib_fp:tht_vertical_rca" H 1275 1550 50  0001 C CNN
 F 3 " ~" H 1275 1550 50  0001 C CNN
 	1    1275 1550
@@
 F 0 "U1" H 3400 2017 50  0000 C CNN
 F 1 "AD8044" H 3400 1926 50  0000 C CNN
-F 2 "Package_DIP:DIP-14_W7.62mm_LongPads" H 3400 1650 50  0001 C CNN
+F 2 "project_parts:DIP+SOIC_14" H 3400 1650 50  0001 C CNN
 F 3 "https://www.analog.com/media/en/technical-documentation/data-sheets/ADA4807-1_4807-2_4807-4.pdf" H 3400 1650 50  0001 C CNN
 	1    3400 1650
@@
 F 0 "U1" H 5600 3108 50  0000 C CNN
 F 1 "AD8044" H 5600 3199 50  0000 C CNN
-F 2 "Package_DIP:DIP-14_W7.62mm_LongPads" H 5600 3475 50  0001 C CNN
+F 2 "project_parts:DIP+SOIC_14" H 5600 3475 50  0001 C CNN
 F 3 "https://www.analog.com/media/en/technical-documentation/data-sheets/ADA4807-1_4807-2_4807-4.pdf" H 5600 3475 50  0001 C CNN
 	3    5600 3475
 	1    0    0    1
 $EndComp
-$Comp
-L Device:R R12
-U 1 1 5EBD119A
-P 5525 3000
-F 0 "R12" V 5318 3000 50  0000 C CNN
-F 1 "1k" V 5409 3000 50  0000 C CNN
-F 2 "Resistor_THT:R_Axial_DIN0207_L6.3mm_D2.5mm_P7.62mm_Horizontal" V 5455 3000 50  0001 C CNN
-F 3 "~" H 5525 3000 50  0001 C CNN
-	1    5525 3000
-	0    1    1    0
-$EndComp
 Text GLabel 5200 3800 0    50   Input ~ 0
 2.5V
@@
 Wire Wire Line
 	5200 3575 5300 3575
-Wire Wire Line
-	5900 3475 5900 3000
-Wire Wire Line
-	5900 3000 5675 3000
 Wire Wire Line
 	5375 3000 5100 3000
@@
 P 8050 1825
 F 0 "U3" H 8200 2775 50  0000 L CNN
-F 1 "4051" H 8200 2675 50  0000 L CNN
+F 1 "CD4051" H 8200 2675 50  0000 L CNN
 F 2 "Package_DIP:DIP-16_W7.62mm_LongPads" H 8050 1825 50  0001 C CNN
 F 3 "http://www.intersil.com/content/dam/Intersil/documents/cd40/cd4051bms-52bms-53bms.pdf" H 8050 1825 50  0001 C CNN
@@
 U 1 1 5EBCD7C2
 P 5550 1375
-F 0 "R3" V 5450 1300 50  0000 C CNN
-F 1 "1k" V 5450 1425 50  0000 C CNN
+F 0 "R3" V 5475 1375 50  0000 C CNN
+F 1 "1.5k" V 5550 1375 50  0000 C CNN
 F 2 "Resistor_THT:R_Axial_DIN0207_L6.3mm_D2.5mm_P7.62mm_Horizontal" V 5480 1375 50  0001 C CNN
 F 3 "~" H 5550 1375 50  0001 C CNN
@@
 F 0 "U1" H 5675 1500 50  0000 C CNN
 F 1 "AD8044" H 5675 1575 50  0000 C CNN
-F 2 "Package_DIP:DIP-14_W7.62mm_LongPads" H 5625 1750 50  0001 C CNN
+F 2 "project_parts:DIP+SOIC_14" H 5625 1750 50  0001 C CNN
 F 3 "https://www.analog.com/media/en/technical-documentation/data-sheets/ADA4807-1_4807-2_4807-4.pdf" H 5625 1750 50  0001 C CNN
 	2    5625 1750
@@
 Connection ~ 5925 1750
 Wire Wire Line
-	5900 3475 6275 3475
-Wire Wire Line
-	6275 3475 6275 1425
-Wire Wire Line
 	6275 1425 7550 1425
 Connection ~ 5900 3475
@@
 F 0 "U1" H 9375 1692 50  0000 C CNN
 F 1 "AD8044" H 9375 1601 50  0000 C CNN
-F 2 "Package_DIP:DIP-14_W7.62mm_LongPads" H 9375 1325 50  0001 C CNN
+F 2 "project_parts:DIP+SOIC_14" H 9375 1325 50  0001 C CNN
 F 3 "https://www.analog.com/media/en/technical-documentation/data-sheets/ADA4807-1_4807-2_4807-4.pdf" H 9375 1325 50  0001 C CNN
 	4    9375 1325
@@
 F 0 "J2" H 10475 1300 50  0000 L CNN
 F 1 "rca" H 10475 1209 50  0000 L CNN
-F 2 "lib_fp:RCJ-024" H 10375 1325 50  0001 C CNN
+F 2 "lib_fp:tht_vertical_rca" H 10375 1325 50  0001 C CNN
 F 3 " ~" H 10375 1325 50  0001 C CNN
 	1    10375 1325
@@
 P 3450 5400
 F 0 "SW1" H 3325 5650 50  0000 C CNN
-F 1 "SW_SPST" H 3350 5550 50  0000 C CNN
+F 1 "SPDT" H 3350 5550 50  0000 C CNN
 F 2 "lib_fp:mini_toggle_switch_tayda" H 3450 5400 50  0001 C CNN
 F 3 "~" H 3450 5400 50  0001 C CNN
@@
 P 3450 5750
 F 0 "SW2" H 3325 6000 50  0000 C CNN
-F 1 "SW_SPST" H 3350 5900 50  0000 C CNN
+F 1 "SPDT" H 3350 5900 50  0000 C CNN
 F 2 "lib_fp:mini_toggle_switch_tayda" H 3450 5750 50  0001 C CNN
 F 3 "~" H 3450 5750 50  0001 C CNN
@@
 Wire Wire Line
 	1250 3825 1250 3625
-$Comp
-L Device:R R1
-U 1 1 5EE653FF
-P 5550 1175
-F 0 "R1" V 5450 1075 50  0000 C CNN
-F 1 "1.5k" V 5450 1225 50  0000 C CNN
-F 2 "Resistor_THT:R_Axial_DIN0207_L6.3mm_D2.5mm_P7.62mm_Horizontal" V 5480 1175 50  0001 C CNN
-F 3 "~" H 5550 1175 50  0001 C CNN
-	1    5550 1175
-	0    1    1    0
-$EndComp
 Wire Wire Line
 	5125 1175 5400 1175
@@
 	5125 1175 5125 1375
 Wire Wire Line
-	5700 1175 5925 1175
-Wire Wire Line
-	5925 1175 5925 1375
-Wire Wire Line
 	5700 1375 5925 1375
-Connection ~ 5925 1375
 Wire Wire Line
 	5925 1375 5925 1750
@@
 F 0 "U1" H 1175 5600 50  0000 C CNN
 F 1 "AD8044" H 1250 5525 50  0000 C CNN
-F 2 "Package_DIP:DIP-14_W7.62mm_LongPads" H 1175 5325 50  0001 C CNN
+F 2 "project_parts:DIP+SOIC_14" H 1175 5325 50  0001 C CNN
 F 3 "https://www.analog.com/media/en/technical-documentation/data-sheets/ADA4807-1_4807-2_4807-4.pdf" H 1175 5325 50  0001 C CNN
 	5    1175 5325
@@
 Wire Wire Line
 	6125 6725 6525 6725
+$Comp
+L Device:R_POT RV5
+U 1 1 605FE70F
+P 5550 1175
+F 0 "RV5" V 5750 1175 50  0000 C CNN
+F 1 "1k_trim" V 5550 1175 50  0000 C CNN
+F 2 "lib_fp:tht_vertical_trimpot_3362" H 5550 1175 50  0001 C CNN
+F 3 "~" H 5550 1175 50  0001 C CNN
+	1    5550 1175
+	0    -1   -1   0
+$EndComp
+NoConn ~ 5700 1175
+Wire Wire Line
+	5925 1375 5925 1075
+Wire Wire Line
+	5925 1075 5550 1075
+Wire Wire Line
+	5550 1075 5550 1025
+Connection ~ 5925 1375
+$Comp
+L Device:R_POT RV7
+U 1 1 60634D8A
+P 6050 3475
+F 0 "RV7" V 5935 3475 50  0000 C CNN
+F 1 "1k_trim" V 5844 3475 50  0000 C CNN
+F 2 "lib_fp:tht_vertical_trimpot_3362" H 6050 3475 50  0001 C CNN
+F 3 "~" H 6050 3475 50  0001 C CNN
+	1    6050 3475
+	0    -1   -1   0
+$EndComp
+Wire Wire Line
+	6050 3325 6275 3325
+Wire Wire Line
+	6275 3325 6275 1425
+NoConn ~ 6200 3475
+$Comp
+L Device:C C16
+U 1 1 6064606D
+P 6275 3600
+F 0 "C16" H 6390 3646 50  0000 L CNN
+F 1 "0.001u" H 6390 3555 50  0000 L CNN
+F 2 "Capacitor_THT:C_Disc_D4.7mm_W2.5mm_P5.00mm" H 6313 3450 50  0001 C CNN
+F 3 "~" H 6275 3600 50  0001 C CNN
+	1    6275 3600
+	1    0    0    -1
+$EndComp
+Wire Wire Line
+	6275 3450 6275 3325
+Connection ~ 6275 3325
+$Comp
+L power:GND #PWR052
+U 1 1 6064B833
+P 6275 3750
+F 0 "#PWR052" H 6275 3500 50  0001 C CNN
+F 1 "GND" H 6280 3577 50  0000 C CNN
+F 2 "" H 6275 3750 50  0001 C CNN
+F 3 "" H 6275 3750 50  0001 C CNN
+	1    6275 3750
+	1    0    0    -1
+$EndComp
+$Comp
+L Device:R_POT RV6
+U 1 1 6064BF44
+P 5525 3000
+F 0 "RV6" V 5725 3000 50  0000 C CNN
+F 1 "1k_trim" V 5525 3000 50  0000 C CNN
+F 2 "lib_fp:tht_vertical_trimpot_3362" H 5525 3000 50  0001 C CNN
+F 3 "~" H 5525 3000 50  0001 C CNN
+	1    5525 3000
+	0    -1   -1   0
+$EndComp
+Wire Wire Line
+	5900 2850 5525 2850
+Wire Wire Line
+	5900 2850 5900 3475
+NoConn ~ 5675 3000
+Text Notes 5975 4050 0    50   ~ 0
+rc delay filter
 $EndSCHEMATC
