File: chroma_luma_invert/invert_logic.sch (KiCad schematic (older format))
At the start: 17 parts, among them U1 AD8044

Commit message: newest circuit revisions
Parts:
- R23: value 5k -> 5.1k
- renumbered R7 to R15, R8 to R16, R9 to R17, R10 to R18, R11 to R19, RV1 to RV5, RV2 to RV6, RV3 to RV7
Changed lines of the file:
@@
 P 4300 2500
 AR Path="/61B96B45" Ref="#PWR?"  Part="1"
-AR Path="/61AE3835/61B96B45" Ref="#PWR022"  Part="1"
-F 0 "#PWR022" H 4300 2250 50  0001 C CNN
+AR Path="/61AE3835/61B96B45" Ref="#PWR043"  Part="1"
+F 0 "#PWR043" H 4300 2250 50  0001 C CNN
 F 1 "GND" H 4305 2327 50  0000 C CNN
 F 2 "" H 4300 2500 50  0001 C CNN
@@
 AR Path="/61AE3835/61B96B4B" Ref="R23"  Part="1"
 F 0 "R23" H 4480 2154 50  0000 R CNN
-F 1 "5k" H 4480 2245 50  0000 R CNN
+F 1 "5.1k" H 4480 2245 50  0000 R CNN
 F 2 "Resistor_THT:R_Axial_DIN0207_L6.3mm_D2.5mm_P7.62mm_Horizontal" V 4480 2200 50  0001 C CNN
 F 3 "~" H 4550 2200 50  0001 C CNN
@@
 P 3850 2050
 AR Path="/61B96B51" Ref="R?"  Part="1"
-AR Path="/61AE3835/61B96B51" Ref="R11"  Part="1"
-F 0 "R11" V 3643 2050 50  0000 C CNN
+AR Path="/61AE3835/61B96B51" Ref="R19"  Part="1"
+F 0 "R19" V 3643 2050 50  0000 C CNN
 F 1 "1k" V 3734 2050 50  0000 C CNN
 F 2 "Resistor_THT:R_Axial_DIN0207_L6.3mm_D2.5mm_P7.62mm_Horizontal" V 3780 2050 50  0001 C CNN
@@
 $EndComp
 $Comp
-L Device:R_POT RV2
+L Device:R_POT RV6
 U 1 1 61BA380C
 P 3450 3000
-F 0 "RV2" H 3380 3046 50  0000 R CNN
+F 0 "RV6" H 3380 3046 50  0000 R CNN
 F 1 "??100k_pot" H 3380 2955 50  0000 R CNN
 F 2 "lib_fp:Potentiometer_Vertical_Large" H 3450 3000 50  0001 C CNN
@@
 P 3700 2850
 AR Path="/61BA4659" Ref="R?"  Part="1"
-AR Path="/61AE3835/61BA4659" Ref="R9"  Part="1"
-F 0 "R9" V 3493 2850 50  0000 C CNN
+AR Path="/61AE3835/61BA4659" Ref="R17"  Part="1"
+F 0 "R17" V 3493 2850 50  0000 C CNN
 F 1 "??10k" V 3584 2850 50  0000 C CNN
 F 2 "Resistor_THT:R_Axial_DIN0207_L6.3mm_D2.5mm_P7.62mm_Horizontal" V 3630 2850 50  0001 C CNN
@@
 P 3700 3150
 AR Path="/61BA4B56" Ref="R?"  Part="1"
-AR Path="/61AE3835/61BA4B56" Ref="R10"  Part="1"
-F 0 "R10" V 3493 3150 50  0000 C CNN
+AR Path="/61AE3835/61BA4B56" Ref="R18"  Part="1"
+F 0 "R18" V 3493 3150 50  0000 C CNN
 F 1 "??10k" V 3584 3150 50  0000 C CNN
 F 2 "Resistor_THT:R_Axial_DIN0207_L6.3mm_D2.5mm_P7.62mm_Horizontal" V 3630 3150 50  0001 C CNN
@@
 Connection ~ 3450 3150
 $Comp
-L Device:R_POT RV1
+L Device:R_POT RV5
 U 1 1 61BA749A
 P 2650 3400
-F 0 "RV1" H 2580 3446 50  0000 R CNN
+F 0 "RV5" H 2580 3446 50  0000 R CNN
 F 1 "??k_trim" H 2580 3355 50  0000 R CNN
 F 2 "lib_fp:tht_vertical_trimpot_3362" H 2650 3400 50  0001 C CNN
@@
 P 2500 3150
 AR Path="/61BA7B45" Ref="R?"  Part="1"
-AR Path="/61AE3835/61BA7B45" Ref="R7"  Part="1"
-F 0 "R7" V 2293 3150 50  0000 C CNN
+AR Path="/61AE3835/61BA7B45" Ref="R15"  Part="1"
+F 0 "R15" V 2293 3150 50  0000 C CNN
 F 1 "??k" V 2384 3150 50  0000 C CNN
 F 2 "Resistor_THT:R_Axial_DIN0207_L6.3mm_D2.5mm_P7.62mm_Horizontal" V 2430 3150 50  0001 C CNN
@@
 P 2500 3650
 AR Path="/61BA81CB" Ref="R?"  Part="1"
-AR Path="/61AE3835/61BA81CB" Ref="R8"  Part="1"
-F 0 "R8" V 2293 3650 50  0000 C CNN
+AR Path="/61AE3835/61BA81CB" Ref="R16"  Part="1"
+F 0 "R16" V 2293 3650 50  0000 C CNN
 F 1 "??k" V 2384 3650 50  0000 C CNN
 F 2 "Resistor_THT:R_Axial_DIN0207_L6.3mm_D2.5mm_P7.62mm_Horizontal" V 2430 3650 50  0001 C CNN
@@
 $EndComp
 $Comp
-L power:+5V #PWR016
+L power:+5V #PWR041
 U 1 1 61BA8A62
 P 2150 3050
-F 0 "#PWR016" H 2150 2900 50  0001 C CNN
+F 0 "#PWR041" H 2150 2900 50  0001 C CNN
 F 1 "+5V" H 2165 3223 50  0000 C CNN
 F 2 "" H 2150 3050 50  0001 C CNN
@@
 	2650 3150 2650 3250
 $Comp
-L power:GND #PWR019
+L power:GND #PWR042
 U 1 1 61BAA0BF
 P 2150 3850
-F 0 "#PWR019" H 2150 3600 50  0001 C CNN
+F 0 "#PWR042" H 2150 3600 50  0001 C CNN
 F 1 "GND" H 2155 3677 50  0000 C CNN
 F 2 "" H 2150 3850 50  0001 C CNN
@@
 	4650 4750 4650 4700
 $Comp
-L Device:R_POT RV3
+L Device:R_POT RV7
 U 1 1 61C1C2CA
 P 3650 5950
-F 0 "RV3" H 3580 5996 50  0000 R CNN
+F 0 "RV7" H 3580 5996 50  0000 R CNN
 F 1 "??100k_pot" H 3580 5905 50  0000 R CNN
 F 2 "lib_fp:Potentiometer_Vertical_Large" H 3650 5950 50  0001 C CNN
