File: two_point_one_colorizer/sync_and_burst.sch (KiCad schematic (older format))
At the start: 17 parts, among them SW2 SPDT_slide, U4 CD4013, U5 74HC4538, U6 LM1881, U7 74HC86

Commit message: updates
Connections:
- net at R10.2, R11.2, U4.3 (C)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: no longer U5.5 (~A)
- net at U6.5 (BURST): now also U5.5 (~A)
- no-connect marks 18 -> 17
Changed lines of the file:
@@
 NoConn ~ 6550 2850
-Wire Wire Line
-	5400 3500 5400 3800
-Wire Wire Line
-	5400 3800 6550 3800
-Connection ~ 5400 3500
 Wire Wire Line
 	7550 3900 9400 3900
@@
 Wire Wire Line
 	6050 3700 6550 3700
-NoConn ~ 5050 2200
 $Comp
 L symbol:74HC4538 U5
@@
 	5050 2000 5050 1800
 Connection ~ 5050 2000
+Wire Wire Line
+	5050 2200 5750 2200
+Wire Wire Line
+	5750 2200 5750 3800
+Wire Wire Line
+	5750 3800 6550 3800
 $EndSCHEMATC
