File: two_point_one_colorizer/two_point_one_colorizer.kicad_pcb (KiCad board)
At the start: 2 copper layers, 100 x 100 mm, 93 parts, among them J1 Barrel_Jack, J2 rca, J3 mini-din4, J4 Conn_02x08_Odd_Even, J5 rca, Q1 2N3904, SW1 SPDT_slide, SW2 SPDT_slide, SW3 SPDT, SW4 SPDT, U1 4069, U10 74LS221, U2 LM317, U3 CD4053, U4 CD4013, U5 74HC4538, U6 LM1881, U7 74HC86, U8 LM393, U9 74LS221, Y1 Crystal, Y2 Crystal

Commit message: updates
Parts:
- Y1: value Crystal -> 3.8MHZ_Crystal
- Y2: value Crystal -> 4.4MHZ_Crystal
